File: OpenRX-Gemini/esp32-c3.kicad_sch (KiCad schematic)
At the start: 35 parts, among them U1 ESP32-C3, U2 TLV75533PDQNR, U9 TS2306A 240GF MSM 9_C2976675, X1 CJ17-400001010B20

Commit message: annotate
Other:
- note added: "07/06/2026"
- note added: "1"
- note added: "ESP32-C3 + peripherals"
