File: OpenRX-Gemini/lr1121.kicad_sch (KiCad schematic)
At the start: 24 parts, among them J1 Conn_Coaxial_Small, T1 0900PC16J0042001E, U3 LR1121IMLTRT, U4 RFX2401C, U5 SKY13373-460LF

Commit message: annotate
Other:
- note added: "07/06/2026"
- note added: "1"
- note added: "LR1121 + 2.4/900 matching + LNA/PA + RF switch"
