File: OpenRX-Lite/esp32c3_sx1281_lite.kicad_sch (KiCad schematic)
At the start: 47 parts, among them U1 ESP32-C3, U2 TLV75533PDQNR, U3 SX1281IMLTRT, X1 CJ17-400001010B20

Commit message: feat(OpenRX-Lite): convert to AntAIO antweight battlebot AIO
Extend OpenRX-Lite (ESP32-C3 + SX1281 ELRS RX) into an integrated
1–2S antweight combat-robot controller in the Malenki-Nano style:

- Triple brushed-DC ESC: 3× DRV8212 (U6/U10 drive, U11 weapon)
- 6-axis IMU LSM6DS3TR-C (U2) on the shared radio SPI bus
- Power: TPS63070 buck-boost (+BATT→5V) + TLV75533 LDO (→3V3),
  AON7407 reverse-polarity P-FET
- New footprints/3D: DFN-8, WSON-8, VQFN-15, LGA-14, SOD-923, IND 2.0×1.6
- Add part datasheets (DRV8212, LSM6DS3TR-C, TPS63070, AON7407)
- CHANGELIST.md: verified open/done items
- REVIEW.md: multi-agent pin/datasheet/electrical design review

Co-Authored-By: Claude Opus 4.8 (1M context) <noreply@anthropic.com>
Parts:
- removed AE2: 47948-0001, OpenRX-Shared:ANT-SMD_47948-0001, symbol OpenRX-Shared:47948-0001
- removed C10: 1uF, Capacitor_SMD:C_0201_0603Metric, symbol Device:C
- removed C16, C8: 10uF, Capacitor_SMD:C_0402_1005Metric, symbol Device:C
- removed R2: 10k, Resistor_SMD:R_0201_0603Metric, symbol Device:R
- removed TP4: GND, OpenRX-Shared:SolderPad_1.2x2.0mm, symbol Connector:TestPoint
- removed TP5: BOOT, OpenRX-Shared:SolderPad_1.2x2.0mm, symbol Connector:TestPoint
- removed U2: TLV75533PDQNR, OpenRX-Shared:X2SON-4_L1.0-W1.0-P0.65-TL-EP, symbol OpenRX-Shared:TLV75533PDQNR
- added AE2: 2450AT18A100E, OpenRX-Shared:ANT-SMD_L3.2-W1.6, symbol OpenRX-Shared:2450AT18A100E
- added C18, C29, C30, C36, C43: 100nF, Capacitor_SMD:C_0201_0603Metric, symbol Device:C
- added C32, C33, C34, C38, C42: 22uF, Capacitor_SMD:C_0805_2012Metric, symbol Device:C
- added C35, C37: 10uF, Capacitor_SMD:C_0603_1608Metric, symbol Device:C
- added C40: 1uF, Capacitor_SMD:C_0201_0603Metric, symbol Device:C
- added C41: 10uF, Capacitor_SMD:C_0402_1005Metric, symbol Device:C
- added L6: FTC201612S1R5MBCA, OpenRX-Shared:IND-SMD_L2.0-W1.6, symbol OpenRX-Shared:FTC201612S1R5MBCA
- added Q2: AON7407, OpenRX-Shared:DFN-8_L3.0-W3.0-P0.65-BL, symbol OpenRX-Shared:AON7407
- added R11, R16: 52.3k, Resistor_SMD:R_0201_0603Metric, symbol Device:R
- added R12, R13, R17, R6, R8: 10k, Resistor_SMD:R_0201_0603Metric, symbol Device:R
- added R14, R15: 100k, Resistor_SMD:R_0201_0603Metric, symbol Device:R
- added TP10, TP12, TP8: M+, OpenRX-Shared:SolderPad_1.2x2.0mm, symbol Connector:TestPoint
- added TP11, TP13, TP9: M-, OpenRX-Shared:SolderPad_1.2x2.0mm, symbol Connector:TestPoint
- added TP14: gnd, OpenRX-Shared:SolderPad_1.2x2.0mm, symbol Connector:TestPoint
- added TP15: 5v, OpenRX-Shared:SolderPad_1.2x2.0mm, symbol Connector:TestPoint
- added TP16: S, OpenRX-Shared:SolderPad_1.2x2.0mm, symbol Connector:TestPoint
- added TP6, TP7: B+, OpenRX-Shared:SolderPad_1.2x2.0mm, symbol Connector:TestPoint
- added U10, U11, U6: DRV8212DSGR, OpenRX-Shared:WSON-8_L2.0-W2.0-P0.50-TL-EP, symbol OpenRX-Shared:DRV8212DSGR
- added U2: LSM6DS3TR-C, Package_LGA:LGA-14_3x2.5mm_P0.5mm_LayoutBorder3x4y, symbol OpenRX-Shared:LSM6DS3TR-C
- added U4: TLV75533PDQNR, OpenRX-Shared:X2SON-4_L1.0-W1.0-P0.65-TL-EP, symbol OpenRX-Shared:TLV75533PDQNR
- added U7: NZ9F6V2ST5G, OpenRX-Shared:SOD-923_L0.8-W0.6-LS1.0-RD, symbol OpenRX-Shared:NZ9F6V2ST5G
- added U8: TPS63070RNMR, OpenRX-Shared:VQFN-15_L3.0-W2.5-P0.50-BL, symbol OpenRX-Shared:TPS63070RNMR
- added U9: TS2306A 240GF MSM 9_C2976675, OpenRX-Shared:SW-SMD_4P-L3.0-W2.0-P0.85-LS3.5, symbol OpenRX-Shared:TS2306A240GFMSM9_C2976675
- C15: value 1uF -> 100nF; LCSC C76935 -> C76939; LCSC Part C76935 -> C76939
- TP1: value RX -> TestPoint; footprint OpenRX-Shared:SolderPad_1.2x2.0mm -> TestPoint:TestPoint_Pad_D1.0mm
- TP2: value TX -> TestPoint; footprint OpenRX-Shared:SolderPad_1.2x2.0mm -> TestPoint:TestPoint_Pad_D1.0mm
- TP3: value 5V -> TestPoint; footprint OpenRX-Shared:SolderPad_1.2x2.0mm -> TestPoint:TestPoint_Pad_D1.0mm
Connections:
- net +3V3: now also C18.1, C29.1, C30.1, C40.1, C41.1, C43.1, R6.1, R8.1, U10.7 (MODE), U10.8 (VCC), U11.7 (MODE), U11.8 (VCC), U2.5 (VDDIO), U2.8 (VDD), U4.1 (OUT), U6.7 (MODE), U6.8 (VCC)
- net +5V: now also C37.1, C38.1, R16.2, TP15.1, U4.3 (EN), U4.4 (IN), U8.7 (Vout); no longer TP3.1
- net BOOT: now also TP3.1, U9.1
- net CHIP_EN: now also U3.3 (NRESET)
- net GND: now also C18.2, C29.2, C30.2, C32.2, C33.2, C34.2, C35.2, C36.1, C37.2, C38.2, C40.2, C41.2, C42.2, C43.2, R12.1, R13.1, R14.2, R17.1, TP14.1, TP7.1, U10.4 (GND), U10.9 (EP), U11.4 (GND), U11.6 (IN1/PH), U11.9 (EP), U2.2 (SDx), U2.3 (SCx), U2.6 (GND), U2.7 (GND), U4.2 (GND), U4.5 (EP), U6.4 (GND), U6.9 (EP), U8.10 (PGND), U8.15 (Vsel), U8.4 (GND), U8.6 (FB2), U9.2; no longer U1.16 (GPIO10)
- net MISO: now also U2.1 (SDO/SA0)
- net MOSI: now also U2.14 (SDA)
- net NSS: now also R6.2
- net SCK: now also U2.13 (SCL)
- net at FL1.3 (OUT): now also AE2.1
- net RIGHT_EN: now reaches TP1.1
- net RIGHT_EN: now also U1.28 (U0TXD), U10.5 (IN2/EN); no longer U1.27 (U0RXD)
- net RIGHT_PH: now reaches TP2.1
- net RIGHT_PH: now also U1.27 (U0RXD), U10.6 (IN1/PH); no longer U1.28 (U0TXD)
- net LEFT_PH: now reaches U1.25 (GPIO18)
- net LEFT_PH: now also U6.6 (IN1/PH)
- net LEFT_EN: now reaches U1.26 (GPIO19)
- net LEFT_EN: now also U6.5 (IN2/EN)
- net VSENSE: now reaches U1.4 (XTAL_32K_P)
- net VSENSE: now also R11.1, R12.2
- net RST renamed IMU_CS
- net IMU_CS: now also R8.2, U2.12 (CS); no longer U3.3 (NRESET)
- new net: Q2.1 (S), Q2.2 (S), Q2.3 (S), TP6.1, U7.1 (K)
- new net: Q2.4 (G), R13.2, U7.2 (A)
- new net: R14.1, U8.1 (PS/SYNC)
- new net: L6.1, U8.11 (L1)
- new net: R15.1, U8.14 (EN)
- new net: C36.2, U8.3 (Vaux)
- new net: R16.1, R17.2, U8.5 (FB)
- new net: L6.2, U8.9 (L2)
- new net: TP9.1, U6.2 (OUT1)
- new net: TP12.1, U11.3 (OUT2)
- new net: TP8.1, U6.3 (OUT2)
- new net: TP11.1, U10.2 (OUT1)
- new net: TP13.1, U11.2 (OUT1)
- new net: TP10.1, U10.3 (OUT2)
- new net +BATT: C32.1, C33.1, C34.1, C35.1, C42.1, Q2.5 (D), Q2.6 (D), Q2.7 (D), Q2.8 (D), Q2.9 (D), R11.2, R15.2, U10.1 (VM), U11.1 (VM), U6.1 (VM), U8.12 (Vin)
- new net WEAPON_EN: TP16.1, U1.16 (GPIO10), U11.5 (IN2/EN)
- no-connect marks 15 -> 18
Other:
- note added: "BUCK/BOOST"
- note added: "IMU"
- note added: "Motors"
- note removed: "5V -> 3.3V, 238mV@500mA maximum dropout"
- moved on the sheet: AE1, C1, C11, C12, C13, C14, C17, C19, C20, C21, C22, C23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
